File: hardware/luxdmx.kicad_sch (KiCad schematic)
At the start: 93 parts, among them J1 XLR-5 NC5FAH, J2 USB-C, J3 HY931147C, J4 DISP SH9, J5 XLR-5 NC5FAH, J6 EXP SH9, J7 DMX-OUT A, J8 DMX-OUT B, Q1 MMBT3904, Q2 MMBT3904, SW1 BOOT, SW2 RST, U1 ESP32-S3-WROOM-1-N8, U2 W5500, U3 CH340C, U4 SY8089, U5 ISO3086DWR, U6 ISO3086DWR, U7 DP9900M-5V, U8 USBLC6-2SC6, U9 TPS2116DRLR, Y1 25MHz

Commit message: rebrand(hardware): Update schematic - all LumiGate → LuxDMX
Fixed all symbol library references and project metadata:
- Symbol refs: lumigate:* → luxdmx:* (336 instances)
- Project name: lumigate → luxdmx
- Netlist comment: lumigate.net → luxdmx.net
- Title block: LumiGate v4 → LuxDMX v4

Schematic now fully branded for LuxDMX.
Parts:
- C1, C10, C11, C14, C15, C16, C17, C18, C19, C2, C20, C21, C23, C24, C25, C26, C27, C28, C29, C30, C31, C4, C5, C8, C9: symbol lumigate:C__v -> luxdmx:C__v
- C12, C13, C22, C3, C6: symbol lumigate:C -> luxdmx:C
- D1, D7: symbol lumigate:SM712 -> luxdmx:SM712
- D10: symbol lumigate:SMAJ60A__v -> luxdmx:SMAJ60A__v
- D11: symbol lumigate:SMAJ5.0A__v -> luxdmx:SMAJ5.0A__v
- D2, D3, D4, D5, D6: symbol lumigate:LED -> luxdmx:LED
- F1: symbol lumigate:PPTC__v -> luxdmx:PPTC__v
- FB1, FB2, FB3: symbol lumigate:FerriteBead__v -> luxdmx:FerriteBead__v
- J1, J5: symbol lumigate:NC5FAH -> luxdmx:NC5FAH
- J2: symbol lumigate:USB_C -> luxdmx:USB_C
- J3: symbol lumigate:HY931147C -> luxdmx:HY931147C
- J4, J6: symbol lumigate:Conn_JSTSH9 -> luxdmx:Conn_JSTSH9
- J7, J8: symbol lumigate:Conn_JSTSH3 -> luxdmx:Conn_JSTSH3
- L1: symbol lumigate:L -> luxdmx:L
- L2, L3: symbol lumigate:ACM2012-201-2P -> luxdmx:ACM2012-201-2P
- MH1, MH2, MH3, MH4: symbol lumigate:MountingHole -> luxdmx:MountingHole
- PS1, PS2: symbol lumigate:B0505S-1W -> luxdmx:B0505S-1W
- Q1, Q2: symbol lumigate:MMBT3904 -> luxdmx:MMBT3904
- R1, R10, R11, R12, R13, R14, R15, R16, R17, R19, R2, R3, R4, R5, R6, R7, R8: symbol lumigate:R -> luxdmx:R
- R18, R9: symbol lumigate:R__v -> luxdmx:R__v
- SW1, SW2: symbol lumigate:SW_PUSH -> luxdmx:SW_PUSH
- U1: symbol lumigate:ESP32-S3-WROOM-1-N8 -> luxdmx:ESP32-S3-WROOM-1-N8
- U2: symbol lumigate:W5500 -> luxdmx:W5500
- U3: symbol lumigate:CH340C -> luxdmx:CH340C
- U4: symbol lumigate:SY8089 -> luxdmx:SY8089
- U5, U6: symbol lumigate:ISO3086DWR -> luxdmx:ISO3086DWR
- U7: symbol lumigate:DP9900M-5V -> luxdmx:DP9900M-5V
- U8: symbol lumigate:USBLC6-2SC6 -> luxdmx:USBLC6-2SC6
- U9: symbol lumigate:TPS2116 -> luxdmx:TPS2116
- Y1: symbol lumigate:Crystal -> luxdmx:Crystal
Other:
- title: LumiGate v4 - Art-Net/sACN -> isolated DMX gateway -> LuxDMX v4 - Art-Net/sACN -> isolated DMX gateway
