File: hardware/luxdmx.kicad_sch (KiCad schematic)
At the start: 101 parts, among them J1 XLR-5 NC5FAH, J2 USB-C, J3 HY931147C, J4 DISP SH9, J5 XLR-5 NC5FAH, J6 EXP SH9, J7 DMX-OUT A, J8 DMX-OUT B, Q1 MMBT3904, Q2 MMBT3904, SW1 BOOT, SW2 RST, U1 ESP32-S3-WROOM-1-N8, U2 W5500, U3 CH340C, U4 SY8089, U5 ISO3086DWR, U6 ISO3086DWR, U7 DP9900M-5V, U8 USBLC6-2SC6, U9 TPS2116DRLR, Y1 25MHz

Commit message: hw: v5.2 -- native USB, TPS2116 priority mode, 3225 crystal (#80)
* hw: v5.2 -- native USB, TPS2116 priority mode, 3225 crystal

Fixes the two hardware defects the v5.00 first article turned up, and drops the
serial bridge while we're in there. Revision goes to v5.2.

The auto-reset transistors had EN and IO0 on the wrong collectors, so flashing
needed the manual BOOT-button dance and a tool asserting DTR or RTS alone could
yank either line. Rather than swap the collectors, the whole bridge is gone:
U3, Q1, Q2, R6, R7 and C15 removed. USB-C now goes straight to the S3's native
USB-Serial-JTAG on IO19/IO20, which is in ROM and gives us the flashing port,
the console and JTAG for free. esptool resets over USB by itself, so there is
no auto-reset circuit left to mis-wire. Six parts fewer, two fewer part numbers
to source, and UART0 is free now (broken out on J6 pins 8/9).

The PoE to USB handover hung the board. The suspected cause (too little cap on
the USB input) was wrong: MODE and PR1 were tied to GND, which selects the
TPS2116's default "higher voltage wins" mode, and two near-equal 5V sources
make that hunt. It runs in priority mode now, MODE on VIN1 so PoE always wins,
with a 30k/10k PR1 divider putting the switchover at 4.0V. Vsw is high on
purpose: VOUT tracks VIN1 down until the switch actually fires, so 4.0V keeps
the rail well clear of the ~2.8V where the ESP hangs.

Crystal moved from the 2520 to the 3225 package (C9006, CL 12pF, so 18pF C0G
load caps). The 2520 kept going out of stock at JLC, the 3225 is the mainstream
size that is always there. R24 also went to a 714k-stock SKU.

Board is fully routed: 0 unrouted, 0 hard DRC. The schematic was stale (it
still had the CH340), so it is regenerated from the netlist and round-trip
verified against it, 0 diff on real nets. BOM/CPL/gerbers regenerated, all 93
parts sourced against live JLC assembly stock (not LCSC retail, which is a
different pool and had me chasing a phantom shortage).

None of this is valida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
Parts:
- removed C15: 100nF, Capacitor_SMD:C_0402_1005Metric, symbol luxdmx:C__v
- removed Q1, Q2: MMBT3904, Package_TO_SOT_SMD:SOT-23, symbol luxdmx:MMBT3904
- removed R6, R7: 10k, Resistor_SMD:R_0402_1005Metric, symbol luxdmx:R
- removed U3: CH340C, C84681:SOP-16_L10.0-W3.9-P1.27-LS6.0-BL, symbol luxdmx:CH340C
- added R24: 30k, Resistor_SMD:R_0402_1005Metric, symbol luxdmx:R__v
- added R25: 10k, Resistor_SMD:R_0402_1005Metric, symbol luxdmx:R__v
- C12, C13: value 33pF C0G -> 18pF C0G
- R9: symbol luxdmx:R__v -> luxdmx:R
- U1: value ESP32-S3-WROOM-1-N8 -> ESP32-S3-WROOM-1-N8R2; symbol luxdmx:ESP32-S3-WROOM-1-N8 -> luxdmx:ESP32-S3-WROOM-1-N8R2
- Y1: footprint Crystal:Crystal_SMD_2520-4Pin_2.5x2.0mm -> Crystal:Crystal_SMD_3225-4Pin_3.2x2.5mm
Connections:
- net +5V_POE: now also U9.3 (VIN1), U9.5 (MODE), R24.1; no longer U9.6 (VIN2)
- net +5V_USBF: now also U9.6 (VIN2); no longer U9.3 (VIN1)
- net GND: now also R25.2; no longer U9.4 (PR1), U9.5 (MODE)
- net S3_RX: now also J6.9
- net S3_TX: now also J6.8
- net USB_DM: now also U1.13 (IO19)
- net USB_DP: now also U1.14 (IO20)
- removed net EXP_IO19: J6.8, U1.13 (IO19)
- removed net EXP_IO20: J6.9, U1.14 (IO20)
- new net N$4: R24.2, R25.1, U9.4 (PR1)
- no-connect marks 41 -> 34
Other:
- note added: "PoE PD (U7) + 5V priority mux (U9 TPS2116, PoE preferred)"
- note added: "USB-C (J2) + ESD (U8) -> S3 native USB (USB-Serial-JTAG on IO19/IO20)"
- note removed: "PoE PD (U7) + 5V ideal-diode OR-ing (U9 TPS2116)"
- note removed: "U3 CH340 USB-UART + USB-C (J2) + auto-reset"
- moved on the sheet: C10, C11, C12, C13, C14, C16, C17, C18, C19, C20, C21, C22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
