File: hardware/luxdmx.kicad_pcb (KiCad board)
At the start: 4 copper layers, 119 x 79 mm, 97 parts, among them J1 XLR-5 NC5FAH, J2 USB-C, J3 HY931147C, J4 DISP SH9, J5 XLR-5 NC5FAH, J6 EXP SH9, J7 DMX-OUT A, J8 DMX-OUT B, SW1 BOOT, SW2 RST, U1 ESP32-S3-WROOM-1-N8R2, U2 W5500, U4 SY8089, U5 ISO3086DWR, U6 ISO3086DWR, U7 DP9900M-5V, U8 USBLC6-2SC6, U9 TPS2116DRLR, Y1 25MHz

Commit message: hw: v6.0 -- give J4 and J6 the same power pins so a swapped cable stops killing displays
J4 (display) and J6 (expansion) are the same JST SH 9-pin part sitting 9mm apart, so a
cable happily plugs into either one. Their power pins did not agree though:

  J4:  1 = +3V3   2 = GND    3.. = signals
  J6:  1 = +5V    2 = +3V3   3   = GND   4.. = signals

so putting the display on J6 fed it +5V on VCC and +3V3 on GND. That is not a theoretical
hazard, it killed a panel on my bench. The other direction is nasty too: an expansion board
in J4 returns its whole ground current through IO4.

J6 is now 1=+3V3 2=GND 3..8=signals 9=GND, matching J4. Worst case for a mixed-up cable is
now that some 3V3 CMOS signals land in the wrong places, which both sides shrug off. A
display plugged into J6 lands RST on GND and just sits there in reset, dark but fine.

Why J6 and not J4: whichever header moves invalidates its own cables, and re-pinning J4
would have put +5V on every display cable that already exists, so the exact same dead
display with a new cause. J6's pinout only landed in v5.2 and nothing is built against it
yet, so it is the cheap one to change.

Two things fall out of that:

  * +5V is gone from J6. Feed 5V loads from your own supply.
  * pin 9 is a second GND rather than a 7th GPIO, because there is no free non-strapping
    GPIO left on the module (IO3/IO45/IO46 are all strapping pins). An extra return on a
    6-signal 1mm header is the better use anyway, and it is what makes a mis-plugged
    display land RST on ground.

New hard gate, scripts/validate_header_parity.py, wired in as gate 8. It re-checks the
invariant on the board itself every run: fatal if two different rails share a pin position
or a positive rail sits opposite a signal, GND-vs-signal allowed since that is current
limited and no worse than the GPIO-vs-GPIO contention we already accept. Ran it against the
old board first to make sure it actually catches the bug, and it fails on exactly pins 1
and 2.

Re-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
Connections:
- J6 pad 1: +5V -> +3V3
- J6 pad 2: +3V3 -> GND
- J6 pad 3: GND -> EXP_IO35
- J6 pad 4: EXP_IO35 -> EXP_IO36
- J6 pad 5: EXP_IO36 -> EXP_IO37
- J6 pad 6: EXP_IO37 -> EXP_IO48
- J6 pad 7: EXP_IO48 -> S3_TX
- J6 pad 8: S3_TX -> S3_RX
- J6 pad 9: S3_RX -> GND
Routing:
- net +5V: track 164.4 -> 155.1 mm, vias 4 -> 3
- net EXP_IO36: track 32.8 -> 31.8 mm
- net GND: vias 63 -> 64
Other:
- board text added: "LuxDMX v6.0"
- board text added: "LuxDMX v6.0 -- KEY FEATURES"
- board text removed: "LuxDMX v5.2"
- board text removed: "LuxDMX v5.2 -- KEY FEATURES"
Changed lines of the file:
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@@
 	(title_block
 		(title "LuxDMX")
-		(rev "v5.2")
+		(rev "v6.0")
 		(company "luxdmx.org")
 	)
@@
 			(layers "F.Cu" "F.Mask" "F.Paste")
 			(roundrect_rratio 0.25)
-			(net "+5V")
+			(net "+3V3")
 		)
 		(pad "2" smd roundrect
@@
 			(layers "F.Cu" "F.Mask" "F.Paste")
 			(roundrect_rratio 0.25)
-			(net "+3V3")
+			(net "GND")
 		)
 		(pad "3" smd roundrect
@@
 			(layers "F.Cu" "F.Mask" "F.Paste")
 			(roundrect_rratio 0.25)
-			(net "GND")
+			(net "EXP_IO35")
 		)
 		(pad "4" smd roundrect
@@
 			(layers "F.Cu" "F.Mask" "F.Paste")
 			(roundrect_rratio 0.25)
-			(net "EXP_IO35")
+			(net "EXP_IO36")
 		)
 		(pad "5" smd roundrect
@@
 			(layers "F.Cu" "F.Mask" "F.Paste")
 			(roundrect_rratio 0.25)
-			(net "EXP_IO36")
+			(net "EXP_IO37")
 		)
 		(pad "6" smd roundrect
@@
 			(layers "F.Cu" "F.Mask" "F.Paste")
 			(roundrect_rratio 0.25)
-			(net "EXP_IO37")
+			(net "EXP_IO48")
 		)
 		(pad "7" smd roundrect
@@
 			(layers "F.Cu" "F.Mask" "F.Paste")
 			(roundrect_rratio 0.25)
-			(net "EXP_IO48")
+			(net "S3_TX")
 		)
 		(pad "8" smd roundrect
@@
 			(layers "F.Cu" "F.Mask" "F.Paste")
 			(roundrect_rratio 0.25)
-			(net "S3_TX")
+			(net "S3_RX")
 		)
 		(pad "9" smd roundrect
@@
 			(layers "F.Cu" "F.Mask" "F.Paste")
 			(roundrect_rratio 0.25)
-			(net "S3_RX")
+			(net "GND")
 		)
 		(pad "MP" smd roundrect
@@
 		)
 	)
-	(gr_text "LuxDMX v5.2"
+	(gr_text "LuxDMX v6.0"
 		(at 108 160.5 0)
 		(layer "F.SilkS")
@@
 		)
 	)
-	(gr_text "LuxDMX v5.2 -- KEY FEATURES"
+	(gr_text "LuxDMX v6.0 -- KEY FEATURES"
 		(at 134.5 135.4 0)
 		(layer "B.SilkS")
@@
 	)
 	(via
-		(at 136.5 106.5)
+		(at 136.5 105.5)
 		(size 0.6)
 		(drill 0.3)
@@
 	)
 	(via
+		(at 136.5 112.5)
+		(size 0.6)
+		(drill 0.3)
+		(layers "F.Cu" "B.Cu")
+		(locked yes)
+		(net "GND")
+	)
+	(via
 		(at 174.2453 165)
 		(size 0.6)
@@
 	)
 	(via
-		(at 136.5 105.5)
+		(at 136.5 104.5)
 		(size 0.6)
 		(drill 0.3)
@@
 	)
 	(segment
-		(start 136.9855 104.5)
-		(end 137.7317 105.2462)
-		(width 0.4)
-		(layer "F.Cu")
-		(net "+5V")
-	)
-	(segment
 		(start 103.52 130.5)
 		(end 104.26 130.5)
@@
 	)
 	(segment
-		(start 136.5 104.5)
-		(end 136.9855 104.5)
-		(width 0.4)
-		(layer "F.Cu")
-		(net "+5V")
-	)
-	(segment
 		(start 175.047 160.6525)
 		(end 176.2945 161.9)
@@
 	)
 	(via
-		(at 137.7317 105.2462)
-		(size 0.6)
-		(drill 0.3)
-		(layers "F.Cu" "B.Cu")
-		(net "+5V")
-	)
-	(via
 		(at 165.9778 161)
 		(size 0.6)
@@
 	(segment
 		(start 143.4156 110.3082)
-		(end 142.7937 110.3082)
-		(width 0.4)
-		(layer "B.Cu")
-		(net "+5V")
-	)
-	(segment
-		(start 143.4156 110.3082)
 		(end 147.1221 106.6017)
 		(width 0.4)
@@
 	)
 	(segment
-		(start 142.7937 110.3082)
-		(end 137.7317 105.2462)
-		(width 0.4)
-		(layer "B.Cu")
-		(net "+5V")
-	)
-	(segment
 		(start 145.9263 116.4991)
 		(end 143.4156 113.9884)
@@
 	)
 	(segment
-		(start 127.3918 99.9157)
-		(end 134.9761 107.5)
+		(start 127.392 99.916)
+		(end 133.976 106.5)
 		(width 0.2)
 		(layer "F.Cu")
@@
 	)
 	(segment
-		(start 134.9761 107.5)
-		(end 136.5 107.5)
+		(start 133.976 106.5)
+		(end 136.5 106.5)
 		(width 0.2)
 		(layer "F.Cu")
@@
 	)
 	(segment
-		(start 138.3439 104.9268)
-		(end 138.3439 107.0116)
+		(start 138.344 104.927)
+		(end 138.344 106.012)
 		(width 0.2)
 		(layer "F.Cu")
@@
 	)
 	(segment
-		(start 138.3439 107.0116)
-		(end 136.8555 108.5)
+		(start 136.856 107.5)
+		(end 136.5 107.5)
 		(width 0.2)
 		(layer "F.Cu")
@@
 	)
 	(segment
-		(start 136.8555 108.5)
-		(end 136.5 108.5)
+		(start 138.344 106.012)
+		(end 136.856 107.5)
 		(width 0.2)
 		(layer "F.Cu")
@@
 	)
 	(segment
-		(start 128.4786 103.0017)
-		(end 134.9769 109.5)
+		(start 133.977 108.5)
+		(end 136.5 108.5)
 		(width 0.2)
 		(layer "F.Cu")
@@
 	)
 	(segment
-		(start 134.9769 109.5)
-		(end 136.5 109.5)
+		(start 128.479 103.002)
+		(end 133.977 108.5)
 		(width 0.2)
 		(layer "F.Cu")
@@
 	)
 	(segment
-		(start 136.5 110.5)
-		(end 133.9586 110.5)
+		(start 136.5 109.5)
+		(end 132.959 109.5)
 		(width 0.2)
 		(layer "F.Cu")
@@
 	)
 	(segment
-		(start 133.9586 110.5)
-		(end 128.4936 105.035)
+		(start 132.959 109.5)
+		(end 128.494 105.035)
 		(width 0.2)
 		(layer "F.Cu")
@@
 	)
 	(segment
-		(start 136.5 111.5)
-		(end 133.966 111.5)
+		(start 136.5 110.5)
+		(end 132.966 110.5)
 		(width 0.2)
 		(layer "F.Cu")
@@
 	)
 	(segment
-		(start 133.966 111.5)
+		(start 132.966 110.5)
 		(end 129.461 106.995)
 		(width 0.2)
@@
 	)
 	(segment
-		(start 136.5 112.5)
-		(end 134.1093 112.5)
+		(start 133.270999 111.5)
+		(end 133.19 111.581)
 		(width 0.2)
 		(layer "F.Cu")
@@
 	)
 	(segment
-		(start 134.1093 112.5)
-		(end 133.1898 111.5805)
+		(start 119.3328 111.5805)
+		(end 119.3074 111.6059)
 		(width 0.2)
 		(layer "F.Cu")
@@
 	)
 	(segment
-		(start 119.3328 111.5805)
-		(end 119.3074 111.6059)
+		(start 104.97 103.0017)
+		(end 108.704 103.0017)
 		(width 0.2)
 		(layer "F.Cu")
@@
 	)
 	(segment
-		(start 104.97 103.0017)
-		(end 108.704 103.0017)
+		(start 136.5 111.5)
+		(end 133.270999 111.5)
 		(width 0.2)
 		(layer "F.Cu")

Commit message: hw: call it v6, not v6.0
A fresh major has never carried a minor here, it was v3, v4 and v5, so v6.0 was
out of step. HW_VERSION is now "6", and the silk plus the title block revision
follow it. Docstring in hw_version.py spells the rule out: a new major drops the
minor, the first tweak on top of it becomes v6.1.

Silk and docs only. Copper is byte-identical (967 items, 0 in, 0 out), all 8 gates
still pass, gerbers regenerated for the new silk.
Other:
- board text added: "LuxDMX v6"
- board text added: "LuxDMX v6 -- KEY FEATURES"
- board text removed: "LuxDMX v6.0"
- board text removed: "LuxDMX v6.0 -- KEY FEATURES"
Changed lines of the file:
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@@
 	(title_block
 		(title "LuxDMX")
-		(rev "v6.0")
+		(rev "v6")
 		(company "luxdmx.org")
 	)
@@
 		)
 	)
-	(gr_text "LuxDMX v6.0"
+	(gr_text "LuxDMX v6"
 		(at 108 160.5 0)
 		(layer "F.SilkS")
@@
 		)
 	)
-	(gr_text "LuxDMX v6.0 -- KEY FEATURES"
+	(gr_text "LuxDMX v6 -- KEY FEATURES"
 		(at 134.5 135.4 0)
 		(layer "B.SilkS")
