File: hardware-carrier/luxdmx-carrier.kicad_pcb (KiCad board)
At the start: 2 copper layers, 100 x 80 mm, 48 parts, among them U3 - MAX485 Modul MAX3485 DMX1, U4 - MAX485 Modul MAX3485 DMX2, U5 - MAX485 Modul MAX3485 DMX3

Commit message: carrier: damping on the pixel data lines, and a return path that matches the feed
Feedback from mdethmers on the forum, measured rather than argued about, and he
was right twice.

The ground return of every pixel output was 2.0 mm against 4.8 on the plus side,
so the return was the limit of the whole rail: 5.3 A against 9.8. That was not
even a geometric constraint - 6.8 mm fits there - it was my own cap, the one
meant for the thin spurs to the bulk capacitor and the buck, applied to the wrong
thing. Now 4.8 mm and 10.1 A, symmetric with the feed.

His other number, 3.5 A for a 4.7 mm track, is IPC-2221 with k=0.024, the
internal-layer constant, at a 10 K rise. This board is two layers, both outer, so
k=0.048 and the same formula gives 9.9 A at 20 K. His "9 mm minimum for 6 A" rule
matches his constant exactly. Both are right, they answer different questions,
and the README now names the assumption instead of only the result.

The data lines had no series damping at all: the 74AHCT541 went straight to the
terminal, switching in 3-5 ns into however much unterminated wire is screwed on.
330 R at each buffer output now, same part as the RS-485 bias so the order does
not grow. Overdamped on purpose - a bit is 300 ns at 800 kHz - and it limits the
current when a data pin meets 5 V or GND.

Measured on the finished board, over 341 mm of data line: 60 % has ground
directly opposite, 31 % has ground alongside within 1.5 mm, 9 % has none in
reach. The last figure is 29 mm in short pieces where the lines cross the supply
bus. Stitching vias would not fix it - a via ties two layers together, it does
not create copper where the pour has been squeezed out - and that is the honest
argument for a fourth layer, not for more vias.

Also here: the W5500 gets 100 nF / 1 uF / 22 uF under the module, ascending away
from its 3V3 pin. The whole board runs off the dev module's 800 mA regulator,
which is enough on current at 269 mA for a full build, but that rail arrives
through 62 mm of 0.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
Parts:
- added 100nF W5500: 100nF, chip-universal, B.Cu at (100.2, 63.5)
- added 1uF W5500: 1uF, chip-universal, B.Cu at (100.2, 68.5)
- added 330R PIX1: 330R pixel, chip-universal, B.Cu at (116.2, 102.0)
- added 330R PIX2: 330R pixel, chip-universal, B.Cu at (124.2, 98.5)
- added 330R PIX3: 330R pixel, chip-universal, B.Cu at (116.2, 95.0)
- added 330R PIX4: 330R pixel, chip-universal, B.Cu at (124.2, 91.5)
- added 330R PIX5: 330R pixel, chip-universal, B.Cu at (116.2, 88.5)
- 22uF W5500: renamed from 100nF; value 100nF -> 22uF W5500
- moved 22uF W5500 7.83 mm to (100.2, 73.5)
- turned 74AHCT541 pixel buffer to 0 degrees
Connections:
- 74AHCT541 pixel buffer pad 14: PIX5_5V -> PIX5_BUF
- 74AHCT541 pixel buffer pad 15: PIX4_5V -> PIX4_BUF
- 74AHCT541 pixel buffer pad 16: PIX3_5V -> PIX3_BUF
- 74AHCT541 pixel buffer pad 17: PIX2_5V -> PIX2_BUF
- 74AHCT541 pixel buffer pad 18: PIX1_5V -> PIX1_BUF
Routing:
- net PIX2_5V: track 56.1 -> 34.1 mm
- net PIX1_5V: track 52.4 -> 30.7 mm
- net PIX4_5V: track 80.9 -> 60.9 mm
- net PIX4_BUF: track 0.00 -> 18.2 mm
- net PIX2_BUF: track 0.00 -> 17.5 mm
- net BTN1: track 99.6 -> 82.3 mm
- net +5V: track 141.8 -> 158.9 mm, vias 3 -> 2
- net PIX3_5V: track 66.3 -> 55.2 mm
- net PIX5_BUF: track 0.00 -> 10.9 mm
- net PIX1_BUF: track 0.00 -> 10.4 mm
- net PIX3_BUF: track 0.00 -> 9.65 mm
- net EXP_IO44: track 81.8 -> 72.4 mm
- net PIX5: track 108.2 -> 116.9 mm, vias 0 -> 1
- net PIX1: track 18.9 -> 27.5 mm
- net I2C_SDA: track 30.1 -> 38.0 mm
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
Commit message: carrier: tie the buffer's unused inputs to GND
A6..A8 on the 74HCT541 (pins 7-9) had no net at all. Floating CMOS
inputs, so extra supply current and the unused outputs can oscillate.
Now one locked 0.4 mm track runs down the pad row to pin 10, which is GND
anyway. tools/tie_unused_buffer_inputs.py does it and is idempotent.

DRC: 0 errors, 0 unconnected, the same 101 silk warnings as before. Only
B_Cu changed in the gerbers, CPL identical. Renders redone with the same
camera as before, near enough.

Boards from the old gerbers: bridge pins 7 to 10 with solder.
Connections:
- 74AHCT541 pixel buffer pad 7: (no net) -> GND
- 74AHCT541 pixel buffer pad 8: (no net) -> GND
- 74AHCT541 pixel buffer pad 9: (no net) -> GND
Routing:
- net GND: track 603.2 -> 607.0 mm
Changed lines of the file:
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@@
 			(layers "B.Cu" "B.Mask" "B.Paste")
 			(roundrect_rratio 0.25)
+			(net "GND")
 		)
 		(pad "8" smd roundrect
@@
 			(layers "B.Cu" "B.Mask" "B.Paste")
 			(roundrect_rratio 0.25)
+			(net "GND")
 		)
 		(pad "9" smd roundrect
@@
 			(layers "B.Cu" "B.Mask" "B.Paste")
 			(roundrect_rratio 0.25)
+			(net "GND")
 		)
 		(pad "10" smd roundrect
@@
 		(layer "B.Cu")
 		(net "GND")
+	)
+	(segment
+		(start 99.235 93.245)
+		(end 99.235 89.435)
+		(width 0.4)
+		(locked yes)
+		(layer "B.Cu")
+		(net "GND")
